File: 回路/SDMDx4/SDMDx4.kicad_pcb (KiCad board)
At the start: 2 copper layers, 147.3 x 96.5 mm, 31 parts, among them J1 Screw_Terminal_01x02, J2 Conn_01x03, J3 Conn_01x03, J4 Conn_01x03, J5 Conn_01x03, J6 Conn_02x12_Odd_Even, J7 Conn_02x12_Odd_Even, J8 Conn_02x12_Odd_Even, J9 Conn_02x12_Odd_Even, U1 74HC00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

Commit message: Add files via upload
Routing:
- net GND: vias 5 -> 8
Changed lines of the file:
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@@
   (segment (start 118.618 110.236) (end 115.062 106.68) (width 1.8) (layer "B.Cu") (net 1))
   (segment (start 122.174 106.68) (end 127 106.68) (width 1.8) (layer "B.Cu") (net 1))
-  (segment (start 154.432 118.872) (end 71.882 118.872) (width 1.8) (layer "F.Cu") (net 2))
+  (segment (start 154.432 118.872) (end 140.97 118.872) (width 1.8) (layer "F.Cu") (net 2))
   (segment (start 71.882 118.872) (end 57.15 118.872) (width 1.8) (layer "F.Cu") (net 2))
+  (segment (start 114.554 118.872) (end 86.614 118.872) (width 1.8) (layer "F.Cu") (net 2))
+  (segment (start 140.97 118.872) (end 114.554 118.872) (width 1.8) (layer "F.Cu") (net 2))
+  (segment (start 86.614 118.872) (end 71.882 118.872) (width 1.8) (layer "F.Cu") (net 2))
   (via (at 127 118.867) (size 0.8) (drill 0.4) (layers "F.Cu" "B.Cu") (net 2))
+  (via (at 114.554 118.872) (size 0.8) (drill 0.4) (layers "F.Cu" "B.Cu") (net 2))
   (via (at 71.882 118.872) (size 0.8) (drill 0.4) (layers "F.Cu" "B.Cu") (net 2))
   (via (at 100.076 118.872) (size 0.8) (drill 0.4) (layers "F.Cu" "B.Cu") (net 2))
   (via (at 57.15 118.872) (size 0.8) (drill 0.4) (layers "F.Cu" "B.Cu") (net 2))
+  (via (at 86.614 118.872) (size 0.8) (drill 0.4) (layers "F.Cu" "B.Cu") (net 2))
+  (via (at 140.97 118.872) (size 0.8) (drill 0.4) (layers "F.Cu" "B.Cu") (net 2))
   (via (at 154.432 118.872) (size 0.8) (drill 0.4) (layers "F.Cu" "B.Cu") (net 2))
   (segment (start 156.972 88.392) (end 166.624 88.392) (width 1.8) (layer "B.Cu") (net 2))
